File: hardware/INA228-V-A-Meter-V2.kicad_pcb (KiCad board)
At the start: 2 copper layers, 75 x 40 mm, 21 parts, among them J1 Banana-Socket, J2 Banana-Socket, J3 Banana-Socket, J4 Banana-Socket, J5 Display-OLED-1.3-Module, U1 SEEEDUINO-XIAO-ESP32C3, U3 INA228

Commit message: Rework PCB
Parts:
- moved H1 15.1 mm to (22.9, 19.9)
- moved H3 15.1 mm to (92.2, 19.9)
Routing:
- net Net-(U3-Vbus): vias 18 -> 0
- net Net-(J3-Pad1): vias 13 -> 0
- net GND: vias 88 -> 93
Other:
- board size 75 x 40 mm -> 75 x 43 mm
