File: hardware/INA228-V-A-Meter.kicad_sch (KiCad schematic)
At the start: 17 parts, among them J1 Banana-Socket, J2 Banana-Socket, J3 Banana-Socket, J4 Banana-Socket, J5 Display-OLED-1.3-Module, U1 SEEEDUINO-XIAO-ESP32C3, U2 LiFePO4-Xiao-Module, U3 INA228

Commit message: Rework PCB
Parts:
- removed U2: LiFePO4-Xiao-Module, Marcus_Modules:LiFePO4-Xiao-Module, symbol Marcus_Modules:LiFePO4-Xiao-Module
- added A1: XIAO-LiFePO4-Power-Module, Marcus_Modules:XIAO-LiFePO4-Power-Module, symbol Marcus_Modules:XIAO-LiFePO4-Power-Module
- added H1, H2, H3, H4: MountingHole_3.4mm, Marcus_Electromechanical:MountingHole_3.2mm_M3, symbol Marcus_Electromechanical:MountingHole_3.2mm
Connections:
- net +3.3V: now also A1.3 (Vout)
- net GND: now also A1.2 (GND)
- net at U1.14 (5V): now also A1.1 (Vin)
- net at U1.1 (PA02_A0_D0): now also A1.5 (Batt_mon)

Commit message: Save
Parts:
- R2, R3: value 10 -> 10R
Changed lines of the file:
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@@
 			)
 		)
-		(property "Value" "10"
+		(property "Value" "10R"
 			(at 83.82 73.66 90)
 			(effects
@@
 			)
 		)
-		(property "Value" "10"
+		(property "Value" "10R"
 			(at 86.36 60.96 90)
 			(effects
