File: hardware/INA228-V-A-Meter.kicad_pcb (KiCad board)
At the start: 2 copper layers, 75 x 40 mm, 21 parts, among them J1 Banana-Socket, J2 Banana-Socket, J3 Banana-Socket, J4 Banana-Socket, J5 Display-OLED-1.3-Module, U1 SEEEDUINO-XIAO-ESP32C3, U3 INA228

Commit message: Save
Parts:
- R2, R3: value 10 -> 10R
- moved H1 15.1 mm to (22.9, 19.9)
- moved H3 15.1 mm to (92.2, 19.9)
Routing:
- net Net-(U3-Vbus): vias 18 -> 0
- net Net-(J3-Pad1): vias 13 -> 0
- net GND: vias 88 -> 93
Other:
- board size 75 x 40 mm -> 75 x 43 mm

Commit message: Rework PCB, Add fabrication and case
Other:
- board text added: "LiPo Battery connection (if LiFePO4 Module not used)"
Changed lines of the file:
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@@
 			(drillshape 0)
 			(scaleselection 1)
-			(outputdirectory "gerbers")
+			(outputdirectory "gerber")
 		)
 	)
@@
 		)
 	)
+	(gr_text "LiPo Battery connection\n(if LiFePO4 Module not used)"
+		(at 80.8 45.2 0)
+		(layer "B.SilkS")
+		(effects
+			(font
+				(size 1 1)
+				(thickness 0.15)
+			)
+			(justify left bottom mirror)
+		)
+	)
